File: Hardware/OpenBook_Schematic.sch (EAGLE design)
At the start: 14 parts, among them IC4 XC6220A331MR-G, J2 SAMACSYS_PARTS_USB4110-GF-A, Q1 20V/4.2A/52mΩ/1.4W

Commit message: added project files
Parts:
- added C1, C10, C2, C6, C8, C9, C_DELAY: 100nF, DeskAssistant v19 v1:ESP32_WROVER_EAGLE-LTSPICE_CC0402
- added C10_SUPERCAP: CPH3225A, DeskAssistant v19 v1:CPH3225A
- added C1_BAT, C2_BAT: 4.7uF, DeskAssistant v19 v1:ESP32_WROVER_EAGLE-LTSPICE_CC0402
- added C4: 4.7uF/25V, DeskAssistant v19 v1:ESP32_WROVER_EAGLE-LTSPICE_CC0402
- added C5: 1uF, DeskAssistant v19 v1:ESP32_WROVER_EAGLE-LTSPICE_CC0402
- added C7: 10uF, DeskAssistant v19 v1:ESP32_WROVER_EAGLE-LTSPICE_CC0402
- added CHANGE_BUTTON, RESET_BUTTON, U$2: BUTTON_CUSYOMV1, DeskAssistant v19 v1:BUTTON_CUSYOMV1
- added CHG_LED: (no value), DeskAssistant v19 v1:ADAFRUIT_LEDCHIP-LED0603
- added D10, D11, D12, D6, D8, D9: PGB1010603MR, DeskAssistant v19 v1:PGB1010603MR
- added D3, D4, D5: MBR0530, DeskAssistant v19 v1:MBR0530
- added D7: ESP32_WROVER_AVX---SD0805S020S1R0_AVX_SD0805S020S1R0_0_0AVX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, DeskAssistant v19 v1:ESP32_WROVER_AVX---SD0805S020S1R0_AVX_SD0805S020S1R0_0_0AVX_SD0805S020S1R0_0_0
- added EPD_C1, EPD_C10, EPD_C11, EPD_C12, EPD_C2, EPD_C6, EPD_C7, EPD_C8, EPD_C9: 1uF/50V, DeskAssistant v19 v1:ESP32_WROVER_EAGLE-LTSPICE_CC0402
- added EPD_C5: 0.1uF/50V, DeskAssistant v19 v1:ESP32_WROVER_EAGLE-LTSPICE_CC0402
- added IC1: BD5229G-TR, DeskAssistant v19 v1:BD5229G-TR
- added J1: FH34SRJ-24S-0.5SH_99_, DeskAssistant v19 v1:FH34SRJ-24S-0.5SH_99_
- added J3: QWIIC_RIGHT_ANGLE, DeskAssistant v19 v1:QWIIC_CONNECTORJS-1MM
- added J4: 112A-TAAR-R03_ATTEND, DeskAssistant v19 v1:112A-TAAR-R03_ATTEND
- added L1: 68uH, DeskAssistant v19 v1:744043680IND_4828-WE-TPC_WRE
- added MCP73831: ESP32_WROVER_SPARKFUN-IC-POWER_MCP73831, DeskAssistant v19 v1:ESP32_WROVER_SPARKFUN-IC-POWER_MCP73831
- added Q2: 20V/4.2A/52mΩ/1.4W, DeskAssistant v19 v1:ESP32_WROVER_SPARKFUN-DISCRETESEMI_MOSFET_PCH-DMG2305UX-7
- added Q3: SI1308EDL-T1-GE3, DeskAssistant v19 v1:SI1308EDL-T1-GE3
- added R1, R10, R1_PINH, R1_PINH1, R2_PINH, R2_PINH1, R4, R5, R6, R7, R8, R9, R_BOOT, R_CHARGE, R_CL1, R_RESET: 10K, DeskAssistant v19 v1:ESP32_WROVER_EAGLE-LTSPICE_RR0402
- added R1_BAT: 200, DeskAssistant v19 v1:ESP32_WROVER_EAGLE-LTSPICE_RR0402
- added R2: 2.2, DeskAssistant v19 v1:ESP32_WROVER_EAGLE-LTSPICE_RR0402
- added R2_BAT: 2K, DeskAssistant v19 v1:ESP32_WROVER_EAGLE-LTSPICE_RR0402
- added R3: 0.47, DeskAssistant v19 v1:ESP32_WROVER_EAGLE-LTSPICE_RR0402
- added R_CAPACITOR: 15, DeskAssistant v19 v1:ESP32_WROVER_EAGLE-LTSPICE_RR0402
- added SENSOR2: ESP32_WROVER_BME680_BME680, DeskAssistant v19 v1:ESP32_WROVER_BME680_BME680
- added SJ1: (no value), DeskAssistant v19 v1:SJ
- added TP1, TP10, TP11, TP12, TP13, TP14, TP15, TP16, TP17, TP2, TP3, TP4, TP5, TP6, TP7, TP8, TP9: TPTP20R, DeskAssistant v19 v1:TPTP20R
- added U1: W25Q512JVEIQ, DeskAssistant v19 v1:W25Q512JVEIQ
- added U2: ESP32-C6-WROOM-1-N8, DeskAssistant v19 v1:ESP32-C6-WROOM-1-N8
- added U3: DS3231SN#, DeskAssistant v19 v1:DS3231SN#
- added U4: MAX17048G+T10, DeskAssistant v19 v1:MAX17048G+T10
Connections:
- new net 32KHZ: R2_PINH1.1, U2.IO1, U3.32KHZ
- new net EPD_3V3: C7.1, EPD_C5.2, J1.15, J1.16, L1.2, Q2.S, TP17.TP
- new net EPD_3V3_C: Q2.G, R_CL1.1, TP13.TP, U2.IO20
- new net EPD_BUSY: J1.9, TP9.TP, U2.IO3
- new net EPD_CS: D6.2, J1.12, R9.1, TP10.TP, U2.IO10
- new net EPD_DC: J1.11, TP11.TP, U2.IO5
- new net EPD_RST: J1.10, TP12.TP, U2.IO23
- new net FLASH_CS: D9.2, R5.1, U1.!CS, U2.IO11
- new net GDR: J1.2, Q3.G, R4.2
- new net GPIO8: R1.1, U2.IO8
- new net I2C_PW: C1.1, C2.1, R1_PINH.2, R2_PINH.2, SENSOR2.CSB, SENSOR2.VDD, SENSOR2.VDDIO, U2.IO19
- new net INT_RTC: R1_PINH1.1, TP15.TP, U2.IO0, U3.SQW/!INT
- new net IO/BOOT: C6.1, R_BOOT.1, U$2.3, U$2.4, U2.IO9
- new net IO/CHARGE: C10.1, CHANGE_BUTTON.3, CHANGE_BUTTON.4, R_CHARGE.1, U2.IO15
- new net MISO: D12.2, J4.DAT0, R8.1, TP6.TP, U1.DO(IO1), U2.IO2
- new net MOSI: D11.2, J1.14, J4.CMD, R7.1, TP7.TP, U1.DI(IO0), U2.IO7
- new net N$10: EPD_C10.2, J1.22
- new net N$11: EPD_C8.2, J1.20
- new net N$12: D7.CATHODE, R_CAPACITOR.1
- new net N$13: EPD_C7.2, J1.19
- new net N$14: EPD_C6.2, J1.18
- new net N$22: EPD_C2.2, J1.5
- new net N$23: EPD_C1.2, J1.4
- new net N$3: MCP73831.STAT, R1_BAT.2
- new net N$5: CHG_LED.C, R1_BAT.1
- new net N$6: C4.1, D3.A, D4.K
- new net N$7: EPD_C12.2, J1.24
- new net N$8: MCP73831.PROG, R2_BAT.2
- new net N$9: C_DELAY.1, IC1.CT
- new net PREVGH: D5.K, EPD_C9.2, J1.21
- new net PREVGL: D4.A, EPD_C11.2, J1.23
- new net RESE: J1.3, Q3.S, R3.2
- new net RESE': R2.2, R3.1, SJ1.2
- new net RESET: C5.1, IC1.VOUT, RESET_BUTTON.3, RESET_BUTTON.4, R_RESET.1, U2.EN
- new net RTC_RST: U2.IO18, U3.!RST
- new net RX: TP2.TP, U2.RXD0/GPIO17
- new net SCK: D10.2, J1.13, J4.CLK, R6.1, TP8.TP, U1.CLK, U2.IO6
- new net SCL: J3.4, R2_PINH.1, SENSOR2.SCK, U2.IO22, U3.SCL, U4.SCL
- new net SDA: J3.3, R1_PINH.1, SENSOR2.SDI, U2.IO21, U3.SDA, U4.SDA
- new net SRC: C4.2, D5.A, L1.1, Q3.D
- new net SS_SD: D8.2, J4.CD/DAT3, R10.1, U2.IO4
- new net TX: TP1.TP, U2.TXD0/GPIO16
- new net VRTC: C10_SUPERCAP.2, C8.1, R_CAPACITOR.2, U3.VBAT
- net 3V3: now also C9.1, D7.ANODE, IC1.VDD, J3.2, J4.VDD, Q2.D, R1.2, R10.2, R1_PINH1.2, R2_PINH1.2, R5.2, R6.2, R7.2, R8.2, R9.2, R_BOOT.2, R_CHARGE.2, R_CL1.2, R_RESET.2, TP16.TP, U1.!HOLD!/!RESET!(IO3), U1.!WP!(IO2), U1.VCC, U2.3V3, U3.VCC
- net GND: now also C1.2, C10.2, C10_SUPERCAP.1, C1_BAT.2, C2.2, C2_BAT.2, C5.2, C6.2, C7.2, C8.2, C9.2, CHANGE_BUTTON.1, CHANGE_BUTTON.2, C_DELAY.2, D10.1, D11.1, D12.1, D3.K, D6.1, D8.1, D9.1, EPD_C1.1, EPD_C10.1, EPD_C11.1, EPD_C12.1, EPD_C2.1, EPD_C5.1, EPD_C6.1, EPD_C7.1, EPD_C8.1, EPD_C9.1, IC1.GND, J1.17, J1.8, J1.MP1, J1.MP2, J3.1, J4.GND_1, J4.GND_2, J4.GND_3, J4.GND_4, J4.VSS, MCP73831.VSS, R2.1, R2_BAT.1, R4.1, RESET_BUTTON.1, RESET_BUTTON.2, SENSOR2.GND, SENSOR2.SDO, SJ1.1, TP4.TP, TP5.TP, U$2.1, U$2.2, U1.EXP, U1.GND, U2.GND, U3.GND, U4.CTG, U4.EP, U4.GND, U4.QSTRT
- net USB_D+: now also U2.IO13
- net USB_D-: now also U2.IO12
- net VBAT: now also C2_BAT.1, MCP73831.VBAT, TP3.TP, U4.CELL, U4.VDD
- net VBUS: now also C1_BAT.1, CHG_LED.A, MCP73831.VIN, TP14.TP
Other:
- note added: "Battery Charge Level"
- note added: "Display Type Selector"
- note added: "E-Paper Display Header"
- note added: "E-Paper Drive Circuit"
- note added: "EPD Power"
- note added: "ESP32 C6"
- note added: "Environmental Sensor BME688"
- note added: "External NOR Flash 64MB"
- note added: "Li-Po Battery Charging Controller"
- note added: "Qwiic / Stemma QT"
- note added: "RTC Module DS3231SN"
- note added: "SD Card"
- note added: "SPI ESD Protection Lines"
- note added: "Test Pads"
- note added: "Voltage Supervisor + Reset & Boot / IO Button"
- note removed: "DeskAssistant v19"
