File: Hardware/OpenBook.brd (EAGLE design)
At the start: 170.3 x 111.2 mm, 103 parts, among them IC1 BD5229G-TR, IC4 XC6220A331MR-G, J1 FH34SRJ-24S-0.5SH_99_, J2 SAMACSYS_PARTS_USB4110-GF-A, J3 QWIIC_RIGHT_ANGLE, J4 112A-TAAR-R03_ATTEND, Q1 20V/4.2A/52mΩ/1.4W, Q2 20V/4.2A/52mΩ/1.4W, Q3 SI1308EDL-T1-GE3, U1 W25Q512JVEIQ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

Commit message: added 3d models for components; added render images
Parts:
- CHANGE_BUTTON, RESET_BUTTON, U$2: value BUTTON_CUSYOMV1 -> BUTTON_CUSYOMV1BUTTONMODEL
- D10, D11, D12, D6, D8, D9: value PGB1010603MR -> PGB1010603MRCOSTUM
- D3, D4, D5: value MBR0530 -> MBR0530COSTUM
- TP1, TP10, TP11, TP12, TP13, TP14, TP15, TP16, TP17, TP2, TP3, TP4, TP5, TP6, TP7, TP8, TP9: value TPTP20R -> TP
